Commit message: adding to xacro files for more flexibility

File: husky_description/urdf/accessories/husky_ur_accessories.urdf.xacro (robot description, xacro)
@@ -4,7 +4,9 @@
   <xacro:include filename="$(find ur_description)/urdf/ur3.urdf.xacro" />
   <xacro:include filename="$(find ur_description)/urdf/ur10.urdf.xacro" />
-  <arg name="ur3_enabled" default="false"/>
-  <arg name="ur5_enabled" default="false"/>
-  <arg name="ur10_enabled" default="false"/>
+  <!-- CHANGE THESE VALUES DURING INTEGRATION -->
+  <xacro:arg name="ur3_enabled" default="false"/>
+  <xacro:arg name="ur5_enabled" default="true"/>
+  <xacro:arg name="ur10_enabled" default="false"/>
+  <!-- CHANGE THESE VALUES DURING INTEGRATION -->
     <xacro:if value="$(arg ur3_enabled)">
       <!-- Spawn arm -->

File: husky_description/urdf/husky.urdf.xacro (robot description, xacro)
@@ -107,15 +107,4 @@
     </xacro:husky_wheel>
     <xacro:husky_decorate />
-    <xacro:if value="$(arg ur5_enabled)">
-      <xacro:property name="reflect" value="-1" />
-      <!-- Spawn arm -->
-      <xacro:ur5_robot prefix="ur5_arm_" joint_limited="true"/>
-      <!-- Join arm -->
-      <joint name="ur5_arm_base" type="fixed">
-        <parent link="top_plate_link" />
-        <child link="ur5_arm_base_link" />
-        <origin xyz="0.3058 0 0.0065" rpy="0.0 0.0 -1.57" />
-      </joint>
-    </xacro:if>
     <xacro:if value="$(arg laser_enabled)">
       <sick_lms1xx_mount prefix="base" topic="scan"/>

Commit message: adding Arch

File: husky_description/urdf/accessories/husky_ur_accessories.urdf.xacro (robot description, xacro)
@@ -9,4 +9,28 @@
   <xacro:arg name="ur10_enabled" default="false"/>
   <!-- CHANGE THESE VALUES DURING INTEGRATION -->
+    <xacro:macro name="sensor_arch" params="prefix parent size:=510 *origin">
+        <!-- Spawn the sensor arch link -->
+        <link name="$sensor_arch_mount_link">
+             <origin xyz="0 0 0" rpy="0 0 0"/>
+             <visual>
+                 <geometry>
+                     <mesh filename="package://husky_description/meshes/integration_arch.dae" />
+                 </geometry>
+             </visual>
+             <collision>
+                 <origin xyz="0 0 0" rpy="0 0 0"/>
+                 <geometry>
+                     <mesh filename="package://husky_description/meshes/integration_arch.dae" />
+                 </geometry>
+             </collision>
+        </link>
+        <!-- Attach the sensor arch to the top plate -->
+        <joint name="$sensor_arch_mount" type="fixed">
+             <xacro:insert_block name="origin"/>
+             <parent link="$top_plate_link"/>
+             <child link="$sensor_arch_mount_link"/>
+	     <origin xyz="0.0 0 0.0" rpy="0.0 0.0 0.0" />
+        </joint>
+    </xacro:macro>
     <xacro:if value="$(arg ur3_enabled)">
       <!-- Spawn arm -->

Commit message: Making easy to modify xacro files for integrators

File: husky_description/urdf/accessories/husky_ur_accessories.urdf.xacro (robot description, xacro)
@@ -4,13 +4,17 @@
   <xacro:include filename="$(find ur_description)/urdf/ur3.urdf.xacro" />
   <xacro:include filename="$(find ur_description)/urdf/ur10.urdf.xacro" />
-  <!-- CHANGE THESE VALUES DURING INTEGRATION -->
+  <!-- CHANGE BELOW VALUES DURING INTEGRATION -->
   <xacro:arg name="ur3_enabled" default="false"/>
   <xacro:arg name="ur5_enabled" default="true"/>
   <xacro:arg name="ur10_enabled" default="false"/>
-  <!-- CHANGE THESE VALUES DURING INTEGRATION -->
-    <xacro:macro name="sensor_arch" params="prefix parent size:=510 *origin">
-        <!-- Spawn the sensor arch link -->
-        <link name="$sensor_arch_mount_link">
-             <origin xyz="0 0 0" rpy="0 0 0"/>
+  <xacro:property name="ur_origin">
+   <origin xyz="0.28 0 0.0065" rpy="0.0 0.0 -1.57" />
+  </xacro:property>
+  <xacro:property name="arch_origin">
+    <origin xyz="-0.32 0.0 0.0" rpy="0.0 0.0 0.0" />
+  </xacro:property>
+  <!-- CHANGE ABOVE VALUES DURING INTEGRATION -->
+    <!-- Spawn the sensor arch link -->
+      <link name="sensor_arch_mount_link">
              <visual>
                  <geometry>
@@ -19,26 +23,23 @@
              </visual>
              <collision>
-                 <origin xyz="0 0 0" rpy="0 0 0"/>
                  <geometry>
                      <mesh filename="package://husky_description/meshes/integration_arch.dae" />
                  </geometry>
              </collision>
-        </link>
-        <!-- Attach the sensor arch to the top plate -->
-        <joint name="$sensor_arch_mount" type="fixed">
-             <xacro:insert_block name="origin"/>
-             <parent link="$top_plate_link"/>
-             <child link="$sensor_arch_mount_link"/>
-	     <origin xyz="0.0 0 0.0" rpy="0.0 0.0 0.0" />
-        </joint>
-    </xacro:macro>
+    </link>
+    <!-- Attach the sensor arch to the top plate -->
+    <joint name="sensor_arch_mount" type="fixed">
+             <parent link="top_plate_link"/>
+             <child link="sensor_arch_mount_link"/>
+             <xacro:insert_block name="arch_origin" />
+    </joint>
     <xacro:if value="$(arg ur3_enabled)">
       <!-- Spawn arm -->
-      <xacro:ur5_robot prefix="ur3_arm_" joint_limited="true"/>
-      <!-- Join arm NEED TO ADJUST THESE VALUES!! -->
+      <xacro:ur3_robot prefix="ur3_arm_" joint_limited="true"/>
+      <!-- Join arm -->
       <joint name="ur3_arm_base" type="fixed">
         <parent link="top_plate_link" />
         <child link="ur3_arm_base_link" />
-        <origin xyz="0.3058 0 0.0065" rpy="0.0 0.0 -1.57" />
+        <xacro:insert_block name="ur_origin" />
       </joint>
     </xacro:if>
@@ -50,15 +51,15 @@
         <parent link="top_plate_link" />
         <child link="ur5_arm_base_link" />
-        <origin xyz="0.3058 0 0.0065" rpy="0.0 0.0 -1.57" />
+        <xacro:insert_block name="ur_origin" />
       </joint>
     </xacro:if>
     <xacro:if value="$(arg ur10_enabled)">
       <!-- Spawn arm -->
-      <xacro:ur5_robot prefix="ur10_arm_" joint_limited="true"/>
-      <!-- Join arm NEED TO ADJUST THESE VALUES!! -->
+      <xacro:ur10_robot prefix="ur10_arm_" joint_limited="true"/>
+      <!-- Join arm -->
       <joint name="ur10_arm_base" type="fixed">
         <parent link="top_plate_link" />
         <child link="ur10_arm_base_link" />
-        <origin xyz="0.3058 0 0.0065" rpy="0.0 0.0 -1.57" />
+        <xacro:insert_block name="ur_origin" />
       </joint>
     </xacro:if>

Commit message: adding gripper models and more config Xacro

File: husky_description/urdf/accessories/husky_ur_accessories.urdf.xacro (robot description, xacro)
@@ -4,4 +4,6 @@
   <xacro:include filename="$(find ur_description)/urdf/ur3.urdf.xacro" />
   <xacro:include filename="$(find ur_description)/urdf/ur10.urdf.xacro" />
+  <xacro:include filename="$(find robotiq_force_torque_sensor)/urdf/robotiq_fts300.urdf.xacro" />
+  <xacro:include filename="$(find robotiq_s_model_control)/urdf/s_model_open.urdf.xacro" />
   <!-- CHANGE BELOW VALUES DURING INTEGRATION -->
   <xacro:arg name="ur3_enabled" default="false"/>
@@ -11,8 +13,25 @@
    <origin xyz="0.28 0 0.0065" rpy="0.0 0.0 -1.57" />
   </xacro:property>
+  <xacro:arg name="ft_300_enabled" default="true"/>
+  <xacro:arg name="ft_300_parent" default="ur5_arm_wrist_3_link"/>
+  <xacro:arg name="ft_300_prefix" default="UR_1_"/>
+  <xacro:property name="ft_300_origin">
+   <origin xyz="0 0 0.009" rpy="0 0 0">
+  </xacro:property>
+  <xacro:arg name="s_model_enabled" default="false"/>
+  <xacro:arg name="s_model_parent" default="$(arg ft_300_prefix)fts_toolside"/>
+  <xacro:arg name="s_model_prefix" default="UR_1_"/>
   <xacro:property name="arch_origin">
     <origin xyz="-0.32 0.0 0.0" rpy="0.0 0.0 0.0" />
   </xacro:property>
   <!-- CHANGE ABOVE VALUES DURING INTEGRATION -->
+    <xacro:if value="$(arg ft_300_enabled)">
+      <!-- Spawn FT Sensor -->
+      <xacro:robotiq_fts300 prefix="$(arg ft_300_prefix)" parent="$(arg ft_300_parent)" origin="ft_300_origin"/>
+    </xacro:if>
+    <xacro:if value="$(arg s_model_enabled)">
+      <!-- Spawn FT Sensor -->
+      <xacro:robotiq_fts300 prefix="$(arg s_model_prefix)" parent="$(arg s_model_parent)"/>
+    </xacro:if>
     <!-- Spawn the sensor arch link -->
       <link name="sensor_arch_mount_link">

Commit message: spelling mistake fixes

File: husky_description/urdf/accessories/husky_ur_accessories.urdf.xacro (robot description, xacro)
@@ -16,7 +16,4 @@
   <xacro:arg name="ft_300_parent" default="ur5_arm_wrist_3_link"/>
   <xacro:arg name="ft_300_prefix" default="UR_1_"/>
-  <xacro:property name="ft_300_origin">
-   <origin xyz="0 0 0.009" rpy="0 0 0">
-  </xacro:property>
   <xacro:arg name="s_model_enabled" default="false"/>
   <xacro:arg name="s_model_parent" default="$(arg ft_300_prefix)fts_toolside"/>
@@ -28,5 +25,5 @@
     <xacro:if value="$(arg ft_300_enabled)">
       <!-- Spawn FT Sensor -->
-      <xacro:robotiq_fts300 prefix="$(arg ft_300_prefix)" parent="$(arg ft_300_parent)" origin="ft_300_origin"/>
+      <xacro:robotiq_fts300 prefix="$(arg ft_300_prefix)" parent="$(arg ft_300_parent)" />
     </xacro:if>
     <xacro:if value="$(arg s_model_enabled)">

File: robotiq_force_torque_sensor/urdf/robotiq_fts300.urdf.xacro (robot description, xacro)
@@ -1,9 +1,8 @@
 <?xml version="1.0"?>
 <robot xmlns:xacro="http://www.ros.org/wiki/xacro" name="robotiq_fts300">
-    <xacro:macro name="robotiq_fts300" params="parent prefix *origin">
+    <xacro:macro name="robotiq_fts300" params="parent prefix">
         <!-- mount the fts to the robot -->
         <joint name="${prefix}fts_fix" type="fixed" >
-            <!--In most cases origin would be flange adapter plate: <origin xyz="0 0 0.009" rpy="0 0 0"/> /-->
-            <insert_block name="origin" />
+            <origin xyz="0 0 0.009" rpy="0 0 0"/>
             <parent link="${parent}" />
             <child link="${prefix}fts_robotside" />

Commit message: changing xacros to fit

File: husky_description/urdf/accessories/husky_ur_accessories.urdf.xacro (robot description, xacro)
@@ -16,5 +16,5 @@
   <xacro:arg name="ft_300_parent" default="ur5_arm_wrist_3_link"/>
   <xacro:arg name="ft_300_prefix" default="UR_1_"/>
-  <xacro:arg name="s_model_enabled" default="false"/>
+  <xacro:arg name="s_model_enabled" default="true"/>
   <xacro:arg name="s_model_parent" default="$(arg ft_300_prefix)fts_toolside"/>
   <xacro:arg name="s_model_prefix" default="UR_1_"/>
@@ -28,6 +28,6 @@
     </xacro:if>
     <xacro:if value="$(arg s_model_enabled)">
-      <!-- Spawn FT Sensor -->
-      <xacro:robotiq_fts300 prefix="$(arg s_model_prefix)" parent="$(arg s_model_parent)"/>
+      <!-- Spawn S model Gripper -->
+      <xacro:s_model_open prefix="$(arg s_model_prefix)" parent="$(arg s_model_parent)"/>
     </xacro:if>
     <!-- Spawn the sensor arch link -->

File: robotiq_s_gripper/robotiq_s_model_control/urdf/s_model_open.urdf.xacro (robot description, xacro)
@@ -1,12 +1,26 @@
 <?xml version="1.0"?>
 <robot xmlns:xacro="http://www.ros.org/wiki/xacro" name="s_model_open">
-    <xacro:macro name="s_model_open" params="parent prefix *origin">
+    <xacro:macro name="s_model_open" params="parent prefix ">
         <!-- mount the Gripper to the robot -->
         <joint name="${prefix}_s_model_fix" type="fixed" >
-            <!--In most cases origin would be flange adapter plate: <origin xyz="0 0 0.009" rpy="0 0 0"/> /-->
-            <insert_block name="origin" />
+            <origin xyz="0.0 0.0 0.0" rpy="0.0 0.0 0.0"/>
             <parent link="${parent}" />
-            <child link="${prefix}fts_robotside" />
+            <child link="${prefix}s_model_link" />
         </joint>
+        <link name="${prefix}s_model_link">
+            <visual>
+                <origin xyz="0 0 0" rpy="0 0 0" />
+                <geometry>
+                    <mesh filename="package://robotiq_s_model_control/meshes/s_model_open.stl" scale= "0.001 0.001 0.001" />
+                </geometry>
+                <material name="black"/>
+            </visual>
+            <collision>
+                <origin xyz="0 0 0" rpy="0 0 0" />
+                <geometry>
+                    <mesh filename="package://robotiq_s_model_control/meshes/s_model_open.stl" scale= "0.001 0.001 0.001" />
+                </geometry>
+            </collision>
+        </link>
     </xacro:macro>
 </robot>

Commit message: mods

File: husky_description/urdf/accessories/husky_ur_accessories.urdf.xacro (robot description, xacro)
@@ -1,6 +1,6 @@
 <?xml version="1.0"?>
 <robot xmlns:xacro="http://ros.org/wiki/xacro" name="extras">
+  <xacro:include filename="$(find ur_description)/urdf/ur3.urdf.xacro" />
   <xacro:include filename="$(find ur_description)/urdf/ur5.urdf.xacro" />
-  <xacro:include filename="$(find ur_description)/urdf/ur3.urdf.xacro" />
   <xacro:include filename="$(find ur_description)/urdf/ur10.urdf.xacro" />
   <xacro:include filename="$(find robotiq_force_torque_sensor)/urdf/robotiq_fts300.urdf.xacro" />
@@ -31,23 +31,4 @@
       <xacro:s_model_open prefix="$(arg s_model_prefix)" parent="$(arg s_model_parent)"/>
     </xacro:if>
-    <!-- Spawn the sensor arch link -->
-      <link name="sensor_arch_mount_link">
-             <visual>
-                 <geometry>
-                     <mesh filename="package://husky_description/meshes/integration_arch.dae" />
-                 </geometry>
-             </visual>
-             <collision>
-                 <geometry>
-                     <mesh filename="package://husky_description/meshes/integration_arch.dae" />
-                 </geometry>
-             </collision>
-    </link>
-    <!-- Attach the sensor arch to the top plate -->
-    <joint name="sensor_arch_mount" type="fixed">
-             <parent link="top_plate_link"/>
-             <child link="sensor_arch_mount_link"/>
-             <xacro:insert_block name="arch_origin" />
-    </joint>
     <xacro:if value="$(arg ur3_enabled)">
       <!-- Spawn arm -->
@@ -80,3 +61,22 @@
       </joint>
     </xacro:if>
+    <!-- Spawn the sensor arch link -->
+      <link name="sensor_arch_mount_link">
+             <visual>
+                 <geometry>
+                     <mesh filename="package://husky_description/meshes/integration_arch.dae" />
+                 </geometry>
+             </visual>
+             <collision>
+                 <geometry>
+                     <mesh filename="package://husky_description/meshes/integration_arch.dae" />
+                 </geometry>
+             </collision>
+    </link>
+    <!-- Attach the sensor arch to the top plate -->
+    <joint name="sensor_arch_mount" type="fixed">
+             <parent link="top_plate_link"/>
+             <child link="sensor_arch_mount_link"/>
+             <xacro:insert_block name="arch_origin" />
+    </joint>
 </robot>

Commit message: Fine tunning gripper position

File: husky_description/urdf/accessories/husky_ur_accessories.urdf.xacro (robot description, xacro)
@@ -14,5 +14,5 @@
   </xacro:property>
   <xacro:arg name="ft_300_enabled" default="true"/>
-  <xacro:arg name="ft_300_parent" default="ur5_arm_wrist_3_link"/>
+  <xacro:arg name="ft_300_parent" default="ur5_arm_tool0"/> <!-- can also be ur5_arm_ee_link -->
   <xacro:arg name="ft_300_prefix" default="UR_1_"/>
   <xacro:arg name="s_model_enabled" default="true"/>

File: robotiq_force_torque_sensor/urdf/robotiq_fts300.urdf.xacro (robot description, xacro)
@@ -4,5 +4,5 @@
         <!-- mount the fts to the robot -->
         <joint name="${prefix}fts_fix" type="fixed" >
-            <origin xyz="0 0 0.009" rpy="0 0 0"/>
+            <origin xyz="0 0 -0.009" rpy="0 0 0"/>
             <parent link="${parent}" />
             <child link="${prefix}fts_robotside" />

File: robotiq_s_gripper/robotiq_s_model_control/urdf/s_model_open.urdf.xacro (robot description, xacro)
@@ -3,9 +3,30 @@
     <xacro:macro name="s_model_open" params="parent prefix ">
         <!-- mount the Gripper to the robot -->
+        <joint name="${prefix}_s_model_adapter" type="fixed" >
+            <origin xyz="0.0 0.0 0.015" rpy="0.0 0.0 0.0"/>
+	    <parent link="${parent}" />
+            <child link="${prefix}s_model_adapter_link" />
+        </joint>
         <joint name="${prefix}_s_model_fix" type="fixed" >
-            <origin xyz="0.0 0.0 0.0" rpy="0.0 0.0 0.0"/>
-            <parent link="${parent}" />
+            <origin xyz="0.0 0.0 0.018" rpy="1.5708 0.0 -0.7854"/>
+            <parent link="${prefix}s_model_adapter_link" />
             <child link="${prefix}s_model_link" />
         </joint>
+        <link name="${prefix}s_model_adapter_link">
+        <visual>
+         <origin xyz="0 0 0" rpy="0 0 0" />
+         <geometry>
+          <cylinder radius="0.04" length="0.03"/>
+         </geometry>
+         <material name="black"/>
+        </visual>
+         <collision>
+         <origin xyz="0 0 0" rpy="0 0 0"/>
+         <geometry>
+         <cylinder radius="0.04" length="0.03"/>
+         </geometry>
+         <material name="red"/>
+        </collision>
+        </link>
         <link name="${prefix}s_model_link">
             <visual>
@@ -21,4 +42,5 @@
                     <mesh filename="package://robotiq_s_model_control/meshes/s_model_open.stl" scale= "0.001 0.001 0.001" />
                 </geometry>
+                <material name="red"/>
             </collision>
         </link>

Commit message: generalized ur loading

File: husky_description/urdf/accessories/husky_ur_accessories.urdf.xacro (robot description, xacro)
@@ -13,5 +13,5 @@
   </xacro:property>
   <xacro:arg name="ft_300_enabled" default="true"/>
-  <xacro:arg name="ft_300_parent" default="ur5_arm_tool0"/>
+  <xacro:arg name="ft_300_parent" default="ur_arm_tool0"/>
   <xacro:arg name="ft_300_prefix" default="UR_1_"/>
   <xacro:arg name="s_model_enabled" default="true"/>
@@ -32,32 +32,20 @@
     <xacro:if value="$(arg ur3_enabled)">
       <!-- Spawn arm -->
-      <xacro:ur3_robot prefix="ur3_arm_" joint_limited="true"/>
-      <!-- Join arm -->
-      <joint name="ur3_arm_base" type="fixed">
-        <parent link="top_plate_link" />
-        <child link="ur3_arm_base_link" />
-        <xacro:insert_block name="ur_origin" />
-      </joint>
+      <xacro:ur3_robot prefix="ur_arm_" joint_limited="true"/>
     </xacro:if>
     <xacro:if value="$(arg ur5_enabled)">
       <!-- Spawn arm -->
-      <xacro:ur5_robot prefix="ur5_arm_" joint_limited="true"/>
-      <!-- Join arm -->
-      <joint name="ur5_arm_base" type="fixed">
-        <parent link="top_plate_link" />
-        <child link="ur5_arm_base_link" />
-        <xacro:insert_block name="ur_origin" />
-      </joint>
+      <xacro:ur5_robot prefix="ur_arm_" joint_limited="true"/>
     </xacro:if>
     <xacro:if value="$(arg ur10_enabled)">
       <!-- Spawn arm -->
-      <xacro:ur10_robot prefix="ur10_arm_" joint_limited="true"/>
+      <xacro:ur10_robot prefix="ur_arm_" joint_limited="true"/>
+    </xacro:if>
       <!-- Join arm -->
-      <joint name="ur10_arm_base" type="fixed">
+      <joint name="ur_arm_base" type="fixed">
         <parent link="top_plate_link" />
-        <child link="ur10_arm_base_link" />
+        <child link="ur_arm_base_link" />
         <xacro:insert_block name="ur_origin" />
       </joint>
-    </xacro:if>
     <!-- Spawn the sensor arch link -->
       <link name="sensor_arch_mount_link">

Commit message: Cleaned up the s model and the collision is much smaller

File: husky_description/urdf/accessories/husky_ur_accessories.urdf.xacro (robot description, xacro)
@@ -16,8 +16,8 @@
   <xacro:arg name="ft_300_parent" default="ur_arm_tool0"/>
   <xacro:arg name="ft_300_prefix" default="UR_1_"/>
-  <xacro:arg name="s_model_enabled" default="false"/>
+  <xacro:arg name="s_model_enabled" default="true"/>
   <xacro:arg name="s_model_parent" default="$(arg ft_300_prefix)fts_toolside"/>
   <xacro:arg name="s_model_prefix" default="UR_1_"/>
-  <xacro:arg name="c_model_enabled" default="true"/>
+  <xacro:arg name="c_model_enabled" default="false"/>
   <xacro:arg name="c_model_parent" default="$(arg ft_300_prefix)fts_toolside"/>
   <xacro:arg name="c_model_prefix" default="UR_1_"/>

File: robotiq_s_gripper/robotiq_s_model_control/urdf/s_model_open.urdf.xacro (robot description, xacro)
@@ -33,14 +33,12 @@
                 <origin xyz="0 0 0" rpy="0 0 0" />
                 <geometry>
-                    <mesh filename="package://robotiq_s_model_control/meshes/s_model_open.stl" scale= "0.001 0.001 0.001" />
+                    <mesh filename="package://robotiq_s_model_control/meshes/s_model_open.dae" />
                 </geometry>
-                <material name="black"/>
             </visual>
             <collision>
                 <origin xyz="0 0 0" rpy="0 0 0" />
                 <geometry>
-                    <mesh filename="package://robotiq_s_model_control/meshes/s_model_open.stl" scale= "0.001 0.001 0.001" />
+                    <mesh filename="package://robotiq_s_model_control/meshes/s_model_open_collision.stl" />
                 </geometry>
-                <material name="red"/>
             </collision>
         </link>
